File: KiCAD/V_01_00/Proximity_sensor_V_01_00/Prox_sens_V_01_00/Prox_sens_V_01_00.sch (KiCad schematic (older format))
At the start: 39 parts

Commit message: pcb
Parts:
- removed C?: 470p, symbol Device:C
- removed D?: D_Bridge_+-AA, symbol Device:D_Bridge_+-AA
- removed D?: D, symbol Device:D
- removed Q?: BC847, Package_TO_SOT_SMD:SOT-23, symbol Transistor_BJT:BC847
- removed Q?: BT136-500, Package_TO_SOT_THT:TO-220-3_Vertical, symbol Triac_Thyristor:BT136-500
- removed Q?: Q_NPN_EBC, symbol Device:Q_NPN_EBC
- removed R?: 4.7, symbol Device:R
- removed R? (x4): 107k, symbol Device:R
- removed R?: 4.7k, symbol Device:R
- added C3: 470p, Capacitor_SMD:C_0805_2012Metric, symbol Device:C
- added C6: 0.8n, Capacitor_SMD:C_0805_2012Metric, symbol Device:C
- added C7: 1n, Capacitor_SMD:C_0805_2012Metric, symbol Device:C
- added D1: 1N4148W, Diode_SMD:D_0805_2012Metric, symbol Device:D
- added D2: MB6S, Package_TO_SOT_SMD:TO-269AA, symbol Diode_Bridge:MB6S
- added D3: Z0103MN, Package_TO_SOT_SMD:SOT-223, symbol Triac_Thyristor:Z0103MN
- added D4: SMAJ400A, Diode_SMD:D_SMA, symbol Device:D_Zener
- added J4: Prog. Conn, Connector_PinHeader_2.54mm:PinHeader_1x05_P2.54mm_Vertical, symbol Connector_Generic:Conn_01x05
- added Q1: BC850, Package_TO_SOT_SMD:SOT-23, symbol Transistor_BJT:BC850
- added Q2: BF722, Package_TO_SOT_SMD:SOT-223-3_TabPin2, symbol Device:Q_NPN_BCE
- added R1, R2, R3, R5: 107k, Resistor_SMD:R_0805_2012Metric, symbol Device:R
- added R11: 4.7k, Resistor_SMD:R_0805_2012Metric, symbol Device:R
- added R14: 100, Resistor_SMD:R_0805_2012Metric, symbol Device:R
- added R4: 10, Resistor_SMD:R_0805_2012Metric, symbol Device:R
- C1: renamed from C?; footprint (none) -> Capacitor_THT:CP_Radial_D8.0mm_P3.50mm
- C10: renamed from C?; footprint (none) -> Capacitor_Tantalum_SMD:CP_EIA-3216-18_Kemet-A
- C11, C12, C13, C14, C15, C2, C5, C8, C9: renamed from C?; footprint (none) -> Capacitor_SMD:C_0805_2012Metric
- C4: renamed from C?; value 100n -> 0.8n; footprint (none) -> Capacitor_SMD:C_0805_2012Metric
- D5: renamed from D?; footprint (none) -> LED_SMD:LED_0805_2012Metric
- J1: renamed from J?; footprint (none) -> Connector_PinHeader_2.54mm:PinHeader_1x02_P2.54mm_Vertical
- J2: renamed from J?; footprint (none) -> Connector_PinHeader_1.00mm:PinHeader_1x02_P1.00mm_Vertical
- J3: renamed from J?; footprint (none) -> Connector_Custom:Prox_sens
- R10, R12, R13, R15, R16, R17, R8, R9: renamed from R?; footprint (none) -> Resistor_SMD:R_0805_2012Metric
- U1: renamed from U?; footprint (none) -> Package_SO:SOIC-8-1EP_3.9x4.9mm_P1.27mm_EP2.41x3.3mm
- U2: renamed from U?; footprint (none) -> Package_SO:TSSOP-8_4.4x3mm_P0.65mm
- U3: renamed from U?; footprint (none) -> Package_DFN_QFN:QFN-16-1EP_3x3mm_P0.5mm_EP1.75x1.75mm
Connections:
- net +5V: now also J4.1 (Pin_1), R11.1
- net +VSW: now also C6.1, C7.1, D2.3 (+), D3.2 (A2), D3.4 (A4), D4.1 (K), R1.2, R4.2; no longer U1.8 (Vin)
- net GND: now also C4.1, C3.2, C6.2, D1.2 (A), D2.4 (-), D3.1 (A1), D4.2 (A), J4.2 (Pin_2), Q1.2 (E), R14.2
- net SWD_CLK: now also J4.4 (Pin_4)
- net SWD_IO: now also J4.5 (Pin_5)
- net ZeroCrossing: now also Q1.3 (C), R11.2
- net at C4.2, J1.2 (Pin_2): now also D2.1 (~~)
- net at J1.1 (Pin_1): now also D2.2 (~~)
- net at R10.1: now also D3.3 (G)
- net at C1.1, C5.2, R8.2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: now also Q2.3 (E)
- net at R8.1, R9.2: now also Q2.1 (B)
- new net: Q2.2 (C), R4.1, U1.8 (Vin)
- new net: C7.2, R14.1
- new net: D1.1 (K), Q1.1 (B), R5.1
- new net: C3.1, R3.1, R5.2
- new net: R2.1, R3.2
- new net: R1.1, R2.2
- no-connect marks 6 -> 8
Other:
- note added: "Programming connector"
- note removed: "GPO used?\nRF used?"
- note removed: "max current?"
- moved on the sheet: C1, C10, C2, C4, C5, C8, C9, J1, J2, R10, R12, R13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

Commit message: changes
Parts:
- C2, C4, C6, C7: footprint Capacitor_SMD:C_0805_2012Metric -> Capacitor_SMD:C_1206_3216Metric
- J1: footprint Connector_PinHeader_2.54mm:PinHeader_1x02_P2.54mm_Vertical -> Connector_Custom:PinHeader_1x02_P5.08mm_Vertical
- Q2: value BF722 -> STN83003
- R10, R14, R4: footprint Resistor_SMD:R_0805_2012Metric -> Resistor_SMD:R_1206_3216Metric
Changed lines of the file:
@@
 F 0 "J1" H 768 1267 50  0000 C CNN
 F 1 "AC_in" H 768 1176 50  0000 C CNN
-F 2 "Connector_PinHeader_2.54mm:PinHeader_1x02_P2.54mm_Vertical" H 850 1050 50  0001 C CNN
+F 2 "Connector_Custom:PinHeader_1x02_P5.08mm_Vertical" H 850 1050 50  0001 C CNN
 F 3 "~" H 850 1050 50  0001 C CNN
 	1    850  1050
@@
 F 0 "C4" H 1765 1346 50  0000 L CNN
 F 1 "0.8n" H 1765 1255 50  0000 L CNN
-F 2 "Capacitor_SMD:C_0805_2012Metric" H 1688 1150 50  0001 C CNN
+F 2 "Capacitor_SMD:C_1206_3216Metric" H 1688 1150 50  0001 C CNN
 F 3 "~" H 1650 1300 50  0001 C CNN
 	1    1650 1300
@@
 F 0 "C2" V 1248 7350 50  0000 C CNN
 F 1 "470n" V 1339 7350 50  0000 C CNN
-F 2 "Capacitor_SMD:C_0805_2012Metric" H 1538 7200 50  0001 C CNN
+F 2 "Capacitor_SMD:C_1206_3216Metric" H 1538 7200 50  0001 C CNN
 F 3 "~" H 1500 7350 50  0001 C CNN
 	1    1500 7350
@@
 F 0 "R10" V 1743 7350 50  0000 C CNN
 F 1 "10" V 1834 7350 50  0000 C CNN
-F 2 "Resistor_SMD:R_0805_2012Metric" V 1880 7350 50  0001 C CNN
+F 2 "Resistor_SMD:R_1206_3216Metric" V 1880 7350 50  0001 C CNN
 F 3 "~" H 1950 7350 50  0001 C CNN
 	1    1950 7350
@@
 F 0 "C6" H 3415 1546 50  0000 L CNN
 F 1 "0.8n" H 3415 1455 50  0000 L CNN
-F 2 "Capacitor_SMD:C_0805_2012Metric" H 3338 1350 50  0001 C CNN
+F 2 "Capacitor_SMD:C_1206_3216Metric" H 3338 1350 50  0001 C CNN
 F 3 "~" H 3300 1500 50  0001 C CNN
 	1    3300 1500
@@
 F 0 "C7" H 3815 1396 50  0000 L CNN
 F 1 "1n" H 3815 1305 50  0000 L CNN
-F 2 "Capacitor_SMD:C_0805_2012Metric" H 3738 1200 50  0001 C CNN
+F 2 "Capacitor_SMD:C_1206_3216Metric" H 3738 1200 50  0001 C CNN
 F 3 "~" H 3700 1350 50  0001 C CNN
 	1    3700 1350
@@
 F 0 "R14" H 3770 1696 50  0000 L CNN
 F 1 "100" H 3770 1605 50  0000 L CNN
-F 2 "Resistor_SMD:R_0805_2012Metric" V 3630 1650 50  0001 C CNN
+F 2 "Resistor_SMD:R_1206_3216Metric" V 3630 1650 50  0001 C CNN
 F 3 "~" H 3700 1650 50  0001 C CNN
 	1    3700 1650
@@
 F 0 "R4" V 643 5200 50  0000 C CNN
 F 1 "10" V 734 5200 50  0000 C CNN
-F 2 "Resistor_SMD:R_0805_2012Metric" V 780 5200 50  0001 C CNN
+F 2 "Resistor_SMD:R_1206_3216Metric" V 780 5200 50  0001 C CNN
 F 3 "~" H 850 5200 50  0001 C CNN
 	1    850  5200
@@
 P 1150 5400
 F 0 "Q2" H 1341 5446 50  0000 L CNN
-F 1 "BF722" H 1341 5355 50  0000 L CNN
+F 1 "STN83003" H 1341 5355 50  0000 L CNN
 F 2 "Package_TO_SOT_SMD:SOT-223-3_TabPin2" H 1350 5500 50  0001 C CNN
 F 3 "~" H 1150 5400 50  0001 C CNN
