File: KiCAD/V_01_00/Proximity_sensor_V_01_00/Prox_sens_V_01_00/Prox_sens_V_01_00.kicad_pcb (KiCad board)
At the start: 2 copper layers, 55 x 14 mm, 44 parts, among them J1 AC_in, J2 NFC_Coil, J3 ProximitySens, J4 Prog. Conn, Q1 BC850, Q2 BF722, U1 MP103, U2 M24SR02-Y, U3 CY8C4014LQI-421

Commit message: changes
Parts:
- C2, C6, C7: footprint Capacitor_SMD:C_0805_2012Metric -> Capacitor_SMD:C_1206_3216Metric
- C4: footprint Capacitor_SMD:C_0805_2012Metric -> Capacitor_SMD:C_1206_3216Metric; moved to B.Cu
- D5, R17: moved to F.Cu
- J1: footprint Connector_PinHeader_2.54mm:PinHeader_1x02_P2.54mm_Vertical -> Connector_Custom:PinHeader_1x02_P5.08mm_Vertical
- Q2: value BF722 -> STN83003
- R10, R14, R4: footprint Resistor_SMD:R_0805_2012Metric -> Resistor_SMD:R_1206_3216Metric
- moved R17 50.6 mm to (122.2, 87.5), turned to 0 degrees
- moved D5 44.7 mm to (127.5, 88.2), turned to 180 degrees
- moved J3 3.70 mm to (174.0, 94.7)
- moved R10 3.20 mm to (131.9, 98.4)
- moved C1 2.85 mm to (146.7, 91.3)
- moved C11 2.40 mm to (173.4, 92.1)
- moved R11 1.56 mm to (147.4, 98.4)
- moved C7 1.46 mm to (124.1, 97.0)
- moved D3 1.30 mm to (136.1, 92.2)
- moved C2 1.30 mm to (137.5, 98.4)
- moved J1 1.25 mm to (121.5, 95.5)
- moved C4 1.10 mm to (122.5, 87.5)
- moved Q1 0.98 mm to (141.7, 97.7)
- moved R14 0.72 mm to (124.1, 92.3)
- moved C6 0.60 mm to (130.1, 93.1)
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Routing:
- net Net-(R17-Pad2): track 7.92 -> 51.9 mm, vias 1 -> 4
- net Net-(D5-Pad2): track 2.12 -> 6.31 mm
- net Net-(J3-Pad1): track 1.76 -> 5.61 mm
- net Net-(D3-Pad3): track 6.85 -> 10.4 mm
- net +VSW: track 24.4 -> 27.8 mm
- net Net-(C1-Pad1): track 26.9 -> 29.5 mm, vias 2 -> 3
- net GND: track 101.9 -> 104.1 mm, vias 6 -> 5
- net Net-(C11-Pad1): track 4.39 -> 6.48 mm
- net ZeroCrossing: track 25.6 -> 27.4 mm, vias 1 -> 3
- net TriacControl: track 28.0 -> 29.5 mm
- net Net-(C2-Pad1): track 1.84 -> 2.80 mm
- net +5V: track 61.5 -> 60.8 mm
- net Net-(D1-Pad1): track 6.89 -> 7.66 mm
- net Net-(Q2-Pad2): track 25.6 -> 24.8 mm
- net Net-(D2-Pad2): track 2.63 -> 3.15 mm

Commit message: change
Parts:
- moved R17 5.10 mm to (127.3, 87.5)
- moved D5 4.26 mm to (123.3, 87.5), turned to 0 degrees
Routing:
- net Net-(R17-Pad2): track 51.9 -> 46.5 mm
- net Net-(D5-Pad2): track 6.31 -> 2.15 mm
- net GND: track 104.1 -> 106.9 mm
